Commit message: camera config

File: description/camera.xacro (robot description, xacro)
@@ -4,13 +4,24 @@
         <parent link="chassis"/>
         <child link="camera_link"/>
-        <origin xyz="0.305 0 0.08" rpy="0 0 0"/> <!--TODO: need to change to our actual camera location-->
+        <origin xyz="0.305 0 0.08" rpy="0 0 0"/> <!--TODO: need to change to our actual camera location. the 0.005 is because the camera has a thickness-->
     </joint>
     <link name="camera_link">
         <visual>
             <geometry>
-                <box size="0.010 0.03 0.03"/>
+                <box size="0.010 0.03 0.03"/> <!--TODO: change the dimension of the camera if needed to-->
             </geometry>
             <material name="red"/>
         </visual>
+        <!-- Need to add collision if the camera sticks out. Need to add inertia if the camera is not on a fixed point-->
+        <!--
+        <collision>
+            <geometry>
+                <cylinder radius="0.05" length="0.04"/>
+            </geometry>
+        </collision>
+        <xacro:inertial_cylinder mass="0.1" length="0.04" radius="0.05">
+            <origin xyz="0 0 0" rpy="0 0 0"/>
+        </xacro:inertial_cylinder>
+        -->
     </link>
     <joint name="camera_optical_joint" type="fixed">
@@ -27,7 +38,7 @@
             <update_rate>10</update_rate>
             <camera>
-                <horizontal_fov>1.089</horizontal_fov>
+                <horizontal_fov>1.089</horizontal_fov> <!--Fov is in radians-->
                 <image>
-                    <format>R8G8B8</format>
+                    <format>R8G8B8</format> <!--8bit for each Green Blue Red-->
                     <width>640</width>
                     <height>480</height>

Commit message: modified:   description/camera.xacro

File: description/camera.xacro (robot description, xacro)
@@ -4,5 +4,5 @@
         <parent link="chassis"/>
         <child link="camera_link"/>
-        <origin xyz="0.321 0 0.300" rpy="0 0 0"/> <!--TODO: need to change to our actual camera location. the 0.005 is because the camera has a thickness-->
+        <origin xyz="0.811 0 0.300" rpy="0 0 0"/> <!--TODO: need to change to our actual camera location. the 0.005 is because the camera has a thickness-->
     </joint>
     <link name="camera_link">

Commit message: modified:   description/camera.xacro

File: description/camera.xacro (robot description, xacro)
@@ -4,5 +4,5 @@
         <parent link="chassis"/>
         <child link="camera_link"/>
-        <origin xyz="0.811 0 0.300" rpy="0 0 0"/> <!--TODO: need to change to our actual camera location. the 0.005 is because the camera has a thickness-->
+        <origin xyz="0.9835 0 0.315" rpy="0 0 0"/> <!--TODO: need to change to our actual camera location. the 0.005 is because the camera has a thickness-->
     </joint>
     <link name="camera_link">

Commit message: changes camera dimensions and added lidar

File: description/camera.xacro (robot description, xacro)
@@ -4,5 +4,5 @@
         <parent link="chassis"/>
         <child link="camera_link"/>
-        <origin xyz="0.305 0 0.08" rpy="0 0 0"/> <!--TODO: need to change to our actual camera location. the 0.005 is because the camera has a thickness-->
+        <origin xyz="0.9835 0 0.315" rpy="0 0 0"/> <!--TODO: need to change to our actual camera location. the 0.005 is because the camera has a thickness-->
     </joint>
     <link name="camera_link">

File: description/robot.urdf.xacro (robot description, xacro)
@@ -3,4 +3,5 @@
     <xacro:include filename="robot_core.xacro" />
     <xacro:include filename="gazebo_control.xacro" />
-    <xacro:include filename="camear.xacro" />
+    <xacro:include filename="lidar.xacro" />
+    <xacro:include filename="camera.xacro" />
 </robot>

Commit message: added lidar info, depth camera xacro, modify slightly the dimension of the robot

File: description/camera.xacro (robot description, xacro)
@@ -4,5 +4,5 @@
         <parent link="chassis"/>
         <child link="camera_link"/>
-        <origin xyz="0.9835 0 0.315" rpy="0 0 0"/> <!--TODO: need to change to our actual camera location. the 0.005 is because the camera has a thickness-->
+        <origin xyz="0.8 0 0.315" rpy="0 0 0"/> <!--TODO: need to change to our actual camera location. the 0.005 is because the camera has a thickness-->
     </joint>
     <link name="camera_link">
@@ -43,5 +43,5 @@
                 <horizontal_fov>1.089</horizontal_fov> <!--Fov is in radians-->
                 <image>
-                    <format>B8G8R8</format> <!--8bit for each Green Blue Red-->
+                    <format>R8G8B8</format> <!--8bit for each Green Blue Red-->
                     <width>640</width>
                     <height>480</height>
@@ -54,6 +54,4 @@
             <plugin name="camera_controller" filename="libgazebo_ros_camera.so">
                 <frame_name>camera_link_optical</frame_name>
-                <min_depth>0.1</min_depth>
-                <max_depth>100.0</max_depth>
             </plugin>
         </sensor>

File: description/depth_camera.xacro (robot description, xacro)
@@ -1,61 +1,16 @@
 <?xml version="1.0"?>
 <robot xmlns:xacro="http://www.ros.org/wiki/xacro" >
-    <!-- Camera Mount -->
-    <link name="camera_mount">
-        <visual>
-            <geometry>
-                <!--box size="0.1 0.1 0.02"/> <! Adjust size to your needs -->
-                <mesh filename="package://esda_bot/urdf_asterius_v4/fcid_camera_mount.stl" scale="1 1 1"/>
-            </geometry>
-            <material name="grey">
-                <color rgba="0.5 0.5 0.5 1.0"/>
-            </material>
-        </visual>
-        <!-- Need to add collision camera mount sticks out. Need to add inertia if the camera mount is not on a fixed point
-        <collision>
-            <geometry>
-                <box size="0.1 0.1 0.02"/>
-            </geometry>
-        </collision>
-        <inertial>
-            <mass value="0.05"/>
-            <origin xyz="0 0 0" rpy="0 0 0"/>
-            <inertia
-                ixx="0.0001" ixy="0.0" ixz="0.0"
-                iyy="0.0001" iyz="0.0"
-                izz="0.0001"/>
-        </inertial>
-        -->
-    </link>
-    <joint name="camera_mount_joint" type="fixed">
+    <joint name="camera_joint" type="fixed">
         <parent link="chassis"/>
-        <child link="camera_mount"/>
-        <origin xyz="0.305 0 0.07" rpy="0 0 0"/> <!-- TODO: adjust the mount to its actual position on the chassis-->
-    </joint>
-    <!-- Attach camera to the mount instead of directly to chassis -->
-    <joint name="camera_joint" type="fixed">
-        <parent link="camera_mount"/>
         <child link="camera_link"/>
-        <origin xyz="0 0 0.01" rpy="0 0 0"/> <!--Camera is slightly above the mount-->
+        <origin xyz="0.8 0 0.315" rpy="0 0 0"/>
     </joint>
     <link name="camera_link">
         <visual>
             <geometry>
-                <!--<box size="0.010 0.03 0.03"/>  TODO: change the dimension of the camera if needed to-->
-                <mesh filename="package://esda_bot/urdf_asterius_v4/zed2_ip_outer_with_lens_v8__3.stl" scale="1 1 1"/>
+                <box size="0.033 0.175 0.03"/>
             </geometry>
             <material name="red"/>
         </visual>
-        <!-- Need to add collision if the camera sticks out. Need to add inertia if the camera is not on a fixed point-->
-        <!--
-        <collision>
-            <geometry>
-                <cylinder radius="0.05" length="0.04"/>
-            </geometry>
-        </collision>
-        <xacro:inertial_cylinder mass="0.1" length="0.04" radius="0.05">
-            <origin xyz="0 0 0" rpy="0 0 0"/>
-        </xacro:inertial_cylinder>
-        -->
     </link>
     <joint name="camera_optical_joint" type="fixed">
@@ -67,12 +22,12 @@
     <gazebo reference="camera_link">
         <material>Gazebo/Red</material>
-        <sensor name="camera" type="camera">
+        <sensor name="camera" type="depth">
             <pose> 0 0 0 0 0 0 </pose>
             <visualize>true</visualize>
             <update_rate>10</update_rate>
             <camera>
-                <horizontal_fov>1.089</horizontal_fov> <!--Fov is in radians-->
+                <horizontal_fov>1.089</horizontal_fov>
                 <image>
-                    <format>B8G8R8</format> <!--8bit for each Green Blue Red-->
+                    <format>B8G8R8</format>
                     <width>640</width>
                     <height>480</height>

File: description/lidar.xacro (robot description, xacro)
@@ -4,5 +4,5 @@
         <parent link="chassis"/>
         <child link="laser_frame"/>
-        <origin xyz="0.1 0 0.175" rpy="0 0 0"/>
+        <origin xyz="0.64 0 0.315" rpy="0 0 0"/>
     </joint>
     <link name="laser_frame">

File: description/robot.urdf.xacro (robot description, xacro)
@@ -3,4 +3,6 @@
     <xacro:include filename="robot_core.xacro" />
     <xacro:include filename="gazebo_control.xacro" />
-    <xacro:include filename="camera.xacro" />
+    <!-- <xacro:include filename="lidar.xacro" /> -->
+    <!-- <xacro:include filename="camera.xacro" /> -->
+    <xacro:include filename="depth_camera.xacro" />
 </robot>

File: description/robot_core.xacro (robot description, xacro)
@@ -14,4 +14,7 @@
         <color rgba="0 0 0 1"/>
     </material>
+    <material name="red">
+        <color rgba="1 0 0 1"/>
+    </material>
     <!-- BASE LINK -->
     <link name="base_link">
@@ -21,11 +24,11 @@
         <parent link="base_link"/>
         <child link="chassis"/>
-        <origin xyz="-0.5 0 0"/>    <!-- TODO: change "-0.1" to the distance from the center of two wheels to the back of the bot-->
+        <origin xyz="-0.965423 0 0"/>    <!-- TODO: change "-0.1" to the distance from the center of two wheels to the back of the bot-->
     </joint>
     <link name="chassis">
         <visual>
-            <origin xyz="0.5 0 0.15"/> <!-- TODO: change origin to half the box size (for now assume the bot is a rectangle box)-->
+            <origin xyz="0.4827115 0 0.15"/> <!-- TODO: change origin to half the box size (for now assume the bot is a rectangle box)-->
             <geometry>
-                <box size="1 0.35 0.30"/> <!-- size of the bot [width = 1m, length = 0.35m, height = 0.36m] -->
+                <box size="0.965423 0.35 0.30"/> <!-- size of the bot [width = 1m, length = 0.35m, height = 0.36m] -->
             </geometry>
             <material name="white"/>
@@ -48,5 +51,5 @@
         <parent link="base_link"/>
         <child link="left_wheel"/>
-        <origin xyz="0.322 0.175 0.0025" rpy="-${pi/2} 0 0" /> <!-- TODO: change y offset to how far the wheel from the center -->
+        <origin xyz="0 0.175 0" rpy="-${pi/2} 0 0" /> <!-- TODO: change y offset to how far the wheel from the center -->
         <axis xyz="0 0 1"/>
     </joint>
@@ -74,5 +77,5 @@
         <parent link="base_link"/>
         <child link="right_wheel"/>
-        <origin xyz="0.322 -0.175 0.0025" rpy="${pi/2} 0 0" /> <!-- TODO: change y offset to how far the wheel from the center -->
+        <origin xyz="0 -0.175 0" rpy="${pi/2} 0 0" /> <!-- TODO: change y offset to how far the wheel from the center -->
         <axis xyz="0 0 -1"/>
     </joint>
@@ -100,5 +103,5 @@
         <parent link="chassis"/>
         <child link="caster_wheel"/>
-        <origin xyz="0.24 0 -0.08"/>
+        <origin xyz="0.24 0 -0.0825"/>
     </joint>
     <link name="caster_wheel">
